File: rp2040.kicad_sch (KiCad schematic)
At the start: 28 parts, among them J1 Conn_ARM_SWD_TagConnect_TC203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, SW1 boot, SW2 reset, U1 LM4040DBZ-3, U2 W25Q128JVS, U3 RP2040, Y1 NX3225GA

Commit message: WIP: layout from scratch
Parts:
- added C9: 100n, Capacitor_SMD:C_0402_1005Metric_Pad0.74x0.62mm_HandSolder, symbol Device:C_Small
- C3, C5: value 8pF -> 8p
- C8: value 1uF -> 1u
- J1: value Conn_ARM_SWD_TagConnect_TC2030-NL -> SWD
- SW1, SW2: footprint Button_Switch_SMD:SW_SPST_B3U-1000P -> Button_Switch_SMD:SW_Push_1P1T_XKB_TS-1187A; LCSC Part# C115357 -> C318884
- U2: footprint Package_SO:SOIC-8_5.23x5.23mm_P1.27mm -> Package_SON:WSON-8-1EP_6x5mm_P1.27mm_EP3.4x4.3mm; LCSC Part# (none) -> C190862
- Y1: value NX3225GA -> X322512MSB4SI; LCSC Part# C481407 -> C9002
Connections:
- net +3V3: now also C9.2
- net GND: now also C9.1
Other:
- moved on the sheet: C3, C5, R1, R6, Y1
